File: Rev P/Transconductance Card.sch (EAGLE design)
At the start: 91 parts, among them IC1 74LS07D, IC10 ASSR-1530, IC12 LT1991MS, IC3 ISC0316-SMD, IC4 OP484, IC5 TLC272D, IC6 74LS00D, IC8 7438, IC9 ASSR-1530, Q1 IRF9Z24NPbF, Q2 2N7000, U1 MCP1700T-3302E/TT, X1 H15MLE

Commit message: Partial Board Routing
Need to finish routing power and update schematic power/GND symbols to be consistent with new convention
Parts:
- removed IC12: LT1991MS, linear-technology:LT1991MS
- removed Q2: 2N7000, UL_2N7002:2N7002_SOT23
- added C48, C49, C51: 1n, resistor:C-USC1206
- added C50: 0.1u, resistor:C-USC1210
- added C52, C55, C60: 1u, MeRCIS Lab Parts:CAPACITORC0805
- added C53, C56, C57, C61: 0.1u, MeRCIS Lab Parts:CAPACITORC0805
- added C54, C58: 0.01u, MeRCIS Lab Parts:CAPACITORC0805
- added C59: 1n, MeRCIS Lab Parts:CAPACITORC0805
- added IC2: 74LS00, MeRCIS Lab Parts:74ALS00_QUAD_NANDD
- added U2: IRF9Z24NPbF, UL_IRF9Z24:IRF9Z24SPBF
- C1, C19: value 0.1u -> 1u; device resistor:C-USC1206 -> MeRCIS Lab Parts:CAPACITORC0805
- C10, C3: value 0.1u -> 470u; device resistor:C-USC1206 -> rcl:CPOL-US140CLH-1010
- C11, C14, C16, C20, C4: device resistor:C-USC1206 -> MeRCIS Lab Parts:CAPACITORC0805
- C12: value 1u -> 10u; device resistor:C-USC1206 -> resistor:C-USC1210
- C13, C7, C9: value 0.01u -> 1u; device resistor:C-USC1206 -> MeRCIS Lab Parts:CAPACITORC0805
- C15, C2, C21, C6: value 0.01u -> 0.1u; device resistor:C-USC1206 -> MeRCIS Lab Parts:CAPACITORC0805
- C17, C24: value 1n -> 1u; device resistor:C-USC1206 -> MeRCIS Lab Parts:CAPACITORC0805
- C18: value 0.1u -> 1u; device resistor:C-USC1210 -> MeRCIS Lab Parts:CAPACITORC0805
- C22: value 10u -> 0.01u; device resistor:C-USC1210 -> MeRCIS Lab Parts:CAPACITORC0805
- C23: value 1u -> 0.01u; device resistor:C-USC1206 -> MeRCIS Lab Parts:CAPACITORC0805
- C25: value 470u -> 1u; device resistor1:UCL1V471MNL1GS -> MeRCIS Lab Parts:CAPACITORC0805
- C26: value 470u -> 0.1u; device resistor1:UCL1V471MNL1GS -> MeRCIS Lab Parts:CAPACITORC0805
- C27, C30, C34: device resistor:C-USC1210 -> MeRCIS Lab Parts:CAPACITORC0805
- C28, C32, C36: value 1n -> 0.1u; device resistor:C-USC1206 -> MeRCIS Lab Parts:CAPACITORC0805
- C29: value 1n -> 10u; device resistor:C-USC1206 -> MeRCIS Lab Parts:CAPACITORC0805
- C31: value 1n -> 0.01u; device resistor:C-USC1206 -> MeRCIS Lab Parts:CAPACITORC0805
- C33: value 0.1u -> 0.01u; device resistor:C-USC1210 -> MeRCIS Lab Parts:CAPACITORC0805
- C35: value 0.1u -> 1n; device resistor:C-USC1210 -> MeRCIS Lab Parts:CAPACITORC0805
- C37: value 0.01u -> 1n; device resistor:C-USC1206 -> MeRCIS Lab Parts:CAPACITORC0805
- C38: value 0.01u -> 1n
- C40, C41: device resistor:C-USC1206 -> resistor:C-USC1210
- C42, C43: value 0.1u -> 1n; device resistor:C-USC1210 -> resistor:C-USC1206
- C44, C46: value 1n -> 0.1u; device resistor:C-USC1206 -> resistor:C-USC1210
- C5: value 0.1u -> 10u; device resistor:C-USC1206 -> resistor:C-USC1210
- C8: value 1u -> 0.1u; device resistor:C-USC1206 -> MeRCIS Lab Parts:CAPACITORC0805
- IC1: value 74LS07D -> 74LS00; device 74xx-eu:74LS07D -> MeRCIS Lab Parts:74LS00_QUAD_NANDD
- IC10: value ASSR-1530 -> LT1991MS; device ASSR-1530:ASSR-1530 -> linear-technology:LT1991MS
- IC3: value ISC0316-SMD -> 74LS07D; device SF_ISC03:ISC0316-SMD -> 74xx-eu:74LS07D
- IC4: value OP484 -> TLC272D; device linear:LM324D -> linear:TLC272D; SPICEPREFIX (none) -> I
- IC5: value TLC272D -> OP484; device linear:TLC272D -> linear:LM324D; SPICEPREFIX I -> (none)
- IC6: value 74LS00D -> SF_ISC03_DC_DC16-SMD; device 74xx-us:74LS00D -> MeRCIS Lab Parts:SF_ISC03_DC_DC16-SMD
- IC8: value 7438 -> ASSR-1530; device SN7438:SN7438DR -> MeRCIS Lab Parts:ASSR-1530_SSR
- IC9: device ASSR-1530:ASSR-1530 -> MeRCIS Lab Parts:ASSR-1530_SSR
- Q1: value IRF9Z24NPbF -> 2N7000; device UL_IRF9Z24:IRF9Z24SPBF -> UL_2N7002:2N7002_SOT23
- R1: value 100ohm -> 20k; device resistor:R-US_M1206 -> rcl:POTENTIOMETER_PT_SPIN
- R10, R25: value 330 -> 1k
- R11: value 330 -> 100ohm
- R12: value 9.1k -> 1ohm; device resistor:R-US_M1206 -> resistor:R-US_R2512
- R13: value 20k -> 10k; device rcl:POTENTIOMETER_PT_SPIN -> resistor:R-US_M1206
- R14: value 220 -> 10k
- R15: value 100k -> 10k
- R16: value 100ohm -> 10k
- R17: value 1k -> 10k
- R18: value 1ohm -> 10k; device resistor:R-US_R2512 -> resistor:R-US_M1206
- R2: value 10k -> 100k
- R20, R21, R22: value 10k -> 330
- R23: value 2k -> 330
- R26: value 330 -> 2k
- R3: value 1k -> 220
- R5: value 5k -> 100ohm; device rcl:POTENTIOMETER_PT_SPIN -> resistor:R-US_M1206
- R6: value 10k -> 1k
- R7: value 10k -> 9.1k
- R8: value 1k -> 5k; device resistor:R-US_M1206 -> rcl:POTENTIOMETER_PT_SPIN
- renumbered D4 to D2, U$1 to IC11
Connections:
- removed net N$12: IC4C.+IN, Q2.D, R8.1
- removed net N$35: IC7.AGND
- removed net N$36: IC7.VDD
- new net +3.3V: C24.1, C28.1, C29.1, IC7.VDD, IC7.VREF, U1.VOUT
- new net AGND: C10.-, C12.2, C13.2, C14.2, C15.2, C16.2, C17.2, C18.2, C19.1, C20.2, C21.1, C22.2, C23.1, C26.2, C3.-, C30.2, C32.2, C5.2, C7.2, C8.2, IC4P.V-, IC7.AGND, R8.1
- new net DGND: C1.2, C11.2, C2.2, C24.2, C25.2, C28.2, C29.2, C4.2, C6.2, C9.2, IC1P.GND, IC2P.GND, IC3P.GND, IC6.1, IC6.8, IC7.DGND, R13.1, R14.1, R15.1, U1.GND
- new net N$37: IC4A.-IN, R2.2, R3.1
- new net VDD: C1.1, C11.1, C2.1, C9.1, IC1P.VCC, IC2P.VCC
- net +20V: now also C10.+, C12.1, C13.1, C15.1, C50.1, C51.1, IC10.P1, IC10.P9, R12.2, R9.2; no longer C24.1, C26.1, C4.1, C43.1, C5.1, IC12.P1, IC12.P9, R18.2, R8.2
- net +24V: now also C18.1, C26.1, C3.+, C5.1, C55.1, C56.1, C58.1, C7.1, C8.1, IC10.V+, IC5P.V+, IC6.16; no longer C1.1, C16.1, C25.1, C37.1, C9.1, IC12.V+, IC3.16, IC4P.V+
- net +3V3: now also R26.1; no longer C10.1, C12.1, IC7.VREF, R23.1, U1.VOUT
- net +5V: now also C16.1, C17.1, C25.1, C4.1, C60.1, C61.1, IC3P.VCC, IC4P.V+, IC6.9, IC8.1, IC8.3, R1.1, R16.1, R17.1, R18.1, R23.2, R24.2, R25.1; no longer C11.1, C15.1, C21.1, C23.1, C8.1, IC10.1, IC10.3, IC1P.VCC, IC3.9, IC5P.V+, IC6P.VCC, IC8P.VCC, R10.2, R11.2, R13.1, R2.1, R21.1, R22.1, R3.1
- net -5V: now also C21.2, C23.2, C27.2, C52.2, C53.2, C54.2, IC10.V-, IC5P.V-, IC6.10, R1.2; no longer C13.2, C38.2, C40.2, IC12.V-, IC3.10, IC4P.V-, R13.2
- net 1: now also IC1B.I0, IC1B.I1, IC1C.I0, IC3C.O, R17.2; no longer IC1C.O, IC6B.I0, IC6B.I1, IC6C.I0, R21.2
- net 2: now also IC1A.I0, IC1A.I1, IC1D.I1, IC3B.O, R18.2; no longer IC1B.O, IC6A.I0, IC6A.I1, IC6D.I1, R2.2
- net 3: now also IC1C.I1, IC1D.I0, IC2C.I0, IC2D.I0, IC3A.O, R16.2; no longer IC1A.O, IC6C.I1, IC6D.I0, IC8C.I0, IC8D.I0, R22.2
- net 3&1: now also IC8.2, R20.1; no longer IC9.2, R24.1
- net 3&2: now also IC8.4, R21.1; no longer IC9.4, R25.1
- net ADC-CS: now also IC3D.I; no longer IC1D.I
- net CLK: now also IC3E.I; no longer IC1E.I
- net GND: now also C38.2, C40.2, C48.2, C49.2, C50.2, C51.2, C52.1, C53.1, C54.1, C55.2, C56.2, C57.2, C58.2, C59.2, C60.2, C61.2, IC10.REF, IC8.7; no longer C1.2, C10.2, C11.2, C12.2, C13.1, C14.2, C15.2, C16.2, C17.2, C18.2, C19.1, C20.2, C21.2, C22.2, C23.2, C24.2, C25.2, C26.2, C27.2, C28.2, C29.2, C3.2, C30.2, C31.2, C32.2, C33.2, C38.1, C4.2, C5.2, C6.2, C8.2, C9.2, IC10.7, IC12.REF, IC1P.GND, IC3.1, IC3.8, IC5P.V-, IC6P.GND, IC7.DGND, IC8P.GND, R20.1, R5.1, R6.1, R7.1, U1.GND
- net H-BDG: now also C34.1, C35.1, IC8.5, U2.D; no longer C17.1, C18.1, IC10.5, Q1.D
- net H-EN: now also IC3A.I, R13.2; no longer IC1A.I, R20.2
- net H-NEG: now also IC3B.I, R15.2; no longer IC1B.I, R6.2
- net H-POS: now also IC3C.I, R14.2; no longer IC1C.I, R7.2
- net LOAD_N: now also C47.1, C48.1, IC8.6, IC8.8; no longer C30.1, C31.1, IC9.6, IC9.8
- net LOAD_P: now also C46.1, C49.1, D1.C1A2, IC9.6, IC9.8; no longer C35.1, C36.1, D3.C1A2, IC10.6, IC10.8
- net LSENSE: now also C36.1, C37.1, IC10.M1, IC10.M9, R10.2, R12.1, U2.S; no longer C27.1, C29.1, IC12.M1, IC12.M9, Q1.S, R17.2, R18.1
- net MISO: now also IC3F.O, R26.2; no longer IC1F.O, R23.2
- net N$1: now also D3.C1A2, IC10.OUT; no longer D1.C1A2, IC12.OUT
- net N$10: now also IC4A.+IN; no longer IC5A.+IN
- net N$11: now also IC5C.+IN, Q1.D, R9.1; no longer Q2.S, R12.2, R4.1
- net N$13: now also R11.2, U2.G; no longer Q1.G, R16.2
- net N$14: now also C31.2, IC5D.-IN, R6.2; no longer C2.2, IC4D.-IN, R4.2
- net N$15: now also C33.2, IC5C.OUT, R11.1; no longer C7.2, IC4C.OUT, R16.1
- net N$16: now also C38.1, C40.1, D1.A1; no longer C34.1, C44.1, D3.A1
- net N$17: now also C30.1, IC5D.+IN, R4.2; no longer C3.1, IC4D.+IN, R9.2
- net N$18: now also C32.1, R7.1, R8.2, R8.3; no longer C41.1, R12.1, R5.2, R5.3
- net N$2: now also Q1.S, R6.1, R7.2; no longer IC5A.-IN, R14.1, R15.2
- net N$20: now also C33.1, IC5C.-IN, R10.1; no longer C7.1, IC4C.-IN, R17.1
- net N$21: now also C27.1, R1.3, R2.1; no longer C40.1, R13.3, R15.1
- net N$22: now also C42.1, C44.1, D1.C2; no longer C32.1, C45.1, D3.C2
- net N$23: now also IC1C.O, IC2B.I0, IC2B.I1; no longer IC6C.O, IC8B.I0, IC8B.I1
- net N$24: now also IC1D.O, IC2A.I0, IC2A.I1; no longer IC6D.O, IC8A.I0, IC8A.I1
- net N$25: now also IC2C.O; no longer IC8C.O
- net N$26: now also IC2B.O, R20.2; no longer IC8B.O, R24.2
- net N$27: now also IC2A.O, R21.2; no longer IC8A.O, R25.2
- net N$28: now also IC4A.OUT, R3.2, R4.1; no longer IC5A.OUT, R14.2, R9.1
- net N$29: now also IC2D.O, R22.2; no longer IC8D.O, R26.2
- net N$3: now also IC3D.O, R23.1; no longer IC1D.O, R10.1
- net N$30: now also C39.1, C41.1; no longer C33.1, C46.1
- net N$32: now also C43.1, C45.1; no longer C28.1, C47.1
- net N$33: now also C57.1, D3.A1; no longer C42.1, D1.A1
- net N$34: now also C59.1, D3.C2; no longer C39.1, D1.C2
- net N$4: now also IC3E.O, R24.1; no longer IC1E.O, R11.1
- net N$5: now also Q1.G, R5.1; no longer Q2.G, R1.1
- net N$6: now also IC1B.O, IC2C.I1; no longer IC6B.O, IC8C.I1
- net N$7: now also IC1A.O, IC2D.I1; no longer IC6A.O, IC8D.I1
- net N$8: now also IC3F.I, R25.2; no longer IC1F.I, R3.2
- net N$9: now also C31.1, IC5D.OUT, R5.2; no longer C2.1, IC4D.OUT, R1.2
- net ~3||1: now also IC9.4; no longer IC10.4
- net ~3||2: now also IC9.2, R22.1; no longer IC10.2, R26.1
Other:
- note added: "IC1 Digital Buffer"
- note added: "IC4 Op Amp"
- note added: "IC5 Op Amp"
- note added: "IC6 & IC8 Quad Nand"
- note removed: "IC1"
- note removed: "IC4"
- note removed: "IC5"
- note removed: "IC6"
- note removed: "IC6, IC8"
