File: Rev P/Transconductance Card.sch (EAGLE design)
At the start: 105 parts, among them IC1 74LS00, IC10 LT1991MS, IC11 ADS8319, IC2 74LS00, IC3 74LS07D, IC4 TLC272D, IC5 OP484, IC6 SF_ISC03_DC_DC16-SMD, IC8 ASSR-1530, IC9 ASSR-1530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

Commit message: Board Routing Finished
Need to clean up silkscreen still
Parts:
- U2: device UL_IRF9Z24:IRF9Z24SPBF -> MeRCIS Lab Parts:UL_IRF9Z24_IRF9Z24SPBF
Changed lines of the file:
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@@
 <part name="C27" library="MeRCIS Lab Parts" deviceset="CAPACITOR" device="C0805" package3d_urn="urn:adsk.eagle:package:23617/2" value="0.1u"/>
 <part name="C32" library="MeRCIS Lab Parts" deviceset="CAPACITOR" device="C0805" package3d_urn="urn:adsk.eagle:package:23617/2" value="0.1u"/>
-<part name="U2" library="UL_IRF9Z24" deviceset="IRF9Z24SPBF" device="" value="IRF9Z24NPbF"/>
+<part name="U2" library="MeRCIS Lab Parts" deviceset="UL_IRF9Z24_IRF9Z24SPBF" device="" value="IRF9Z24NPbF"/>
 <part name="D1" library="diode" library_urn="urn:adsk.eagle:library:210" deviceset="BAS70-04" device="" package3d_urn="urn:adsk.eagle:package:43389/2"/>
 <part name="D2" library="diode" library_urn="urn:adsk.eagle:library:210" deviceset="BAS70-04" device="" package3d_urn="urn:adsk.eagle:package:43389/2"/>
